File: ProjectFiles/EAGLE/ECE445_OddsBooster/DataBoard.brd (EAGLE design)
At the start: 100 x 80 mm, 76 parts, among them U2 74LV164D-SHIFT_REGISTER, U3 74LV164D-SHIFT_REGISTER, U4 74LV164D-SHIFT_REGISTER, U5 LP3965-ADJ-LDO, U6 MIC2169-BUCK, U7 S-8337ABIA-T8T1U-BOOSTCONVERT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, U8 MFRC500, X1 FH40-40S-HIROSE-FPC, X2 XH-BAT-CONN, X3 CFPX-180-XTAL-OSCILLATOR

Commit message: PCB done along with generated gerber files
Parts:
- C2: device OddsBooster_3_8_6PM:865080640004-ELECTROLYTIC-CAP -> OddsBooster:865080640004-ELECTROLYTIC-CAP
- X3: device OddsBooster_3_8_6PM:CFPX-180-XTAL-OSCILLATOR -> OddsBooster:CFPX-180-XTAL-OSCILLATOR
- moved L4 106.3 mm to (48.3, 78.1), turned to 270 degrees
- moved AE1 102.6 mm to (55.5, 73.0), turned to 90 degrees
- moved C19 99.2 mm to (15.5, 67.1)
- moved C2 97.3 mm to (23.4, 61.2), turned to 180 degrees
- moved C17 97.0 mm to (27.7, 64.4), turned to 90 degrees
- moved C18 94.2 mm to (14.5, 62.4), turned to 90 degrees
- moved X3 90.4 mm to (44.6, 46.4), turned to 270 degrees
- moved C10 90.0 mm to (48.3, 45.3), turned to 90 degrees
- moved C20 88.6 mm to (11.2, 62.0), turned to 270 degrees
- moved C21 85.3 mm to (29.1, 44.2)
- moved R11 85.1 mm to (28.7, 57.3), turned to 180 degrees
- moved C12 83.8 mm to (23.4, 57.9), turned to 270 degrees
- moved C15 80.9 mm to (38.5, 44.2)
- moved C11 80.7 mm to (33.7, 44.2)
- moved R12 76.0 mm to (23.4, 48.0), turned to 270 degrees
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Routing:
- net N$13: track 0.00 -> 162.5 mm, vias 0 -> 5
- net 0: track 0.00 -> 113.9 mm, vias 0 -> 4
- net VCC: track 261.2 -> 326.6 mm, vias 8 -> 12
- net N$14: track 0.00 -> 63.9 mm
- net D0: track 30.5 -> 59.6 mm
- net N$9: track 0.00 -> 28.7 mm, vias 0 -> 2
- net D1: track 30.3 -> 56.4 mm
- net D4: track 30.5 -> 55.3 mm, vias 2 -> 4
- net D7: track 33.4 -> 58.1 mm, vias 2 -> 4
- net D6: track 33.0 -> 57.7 mm, vias 2 -> 4
- net D5: track 30.9 -> 55.5 mm, vias 2 -> 4
- net ALE: track 11.6 -> 36.2 mm, vias 2 -> 4
- net N$12: track 0.00 -> 23.8 mm, vias 0 -> 2
- net IRQ: track 11.6 -> 35.0 mm
- net D2: track 32.1 -> 55.0 mm
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Other:
- board text added: "C2"
- board text added: "ECE 445 Senior Design Project Lab Odds Booster Team 37"
- board text added: "X3"
- board text removed: "ECE445 Team 37 Odds Booster"

Commit message: working bluetooth mcu firmware, flash-able lcd mcu firmware, working bluetooth app debug and connection window
Parts:
- L2: value 10u -> 3.3u
Changed lines of the file:
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@@
 <attribute name="NAME" x="32.595" y="1.251" size="0.254" layer="25" rot="R180"/>
 </element>
-<element name="L2" library="OddsBooster" package="SRP0415-BOURNS-100K-10U" value="10u" x="39.497" y="2.032" smashed="yes" rot="R90">
+<element name="L2" library="OddsBooster" package="SRP0415-BOURNS-100K-10U" value="3.3u" x="39.497" y="2.032" smashed="yes" rot="R90">
 <attribute name="NAME" x="40.386" y="4.318" size="1.27" layer="25" rot="R180"/>
 </element>
